Commit message: fix warning

File: orne_box_description/urdf/orne_box_3d_lidar.urdf.xacro (robot description, xacro)
@@ -2,4 +2,5 @@
 <robot xmlns:xacro="http://www.ros.org/wiki/xacro" name="orne_box">
   <xacro:arg name="ignition_gazebo" default="false"/>
+  <xacro:arg name="use_camera" default="true"/>
   <xacro:include filename="$(find orne_box_description)/urdf/orne_box.urdf.xacro"/>
   <!-- @TODO More clear boolean operation -->
@@ -80,6 +81,8 @@
   </xacro:sensor_gnss>
   <!-- Setting for Camera -->
-  <xacro:sensor_camera name="camera" parent="base_link">
-    <origin xyz="-0.08 0.0 0.8" rpy="0 0.38 0"/>
-  </xacro:sensor_camera>
+  <xacro:if value="$(arg use_camera)">
+    <xacro:sensor_camera name="camera" parent="base_link">
+      <origin xyz="-0.08 0.0 0.8" rpy="0 0.38 0"/>
+    </xacro:sensor_camera>
+  </xacro:if>
 </robot>

File: orne_box_description/urdf/sensors/camera.urdf.xacro (robot description, xacro)
@@ -19,5 +19,5 @@
           <box size="0.033 0.175 0.03"/>
         </geometry>
-        <material name="bule"/>
+        <material name="blue"/>
       </visual>
     </link>
